Commit message: launch

File: src/dual_ur5/urdf/dual_ur5e.urdf.xacro (robot description, xacro)
@@ -1,11 +1,16 @@
 <?xml version="1.0"?>
 <robot xmlns:xacro="http://wiki.ros.org/xacro" name="dual_ur5e_system">
-    <link name="world"/>
-    <xacro:include filename="$(find ur_description)/urdf/ur_macro.xacro"/>
-    <xacro:arg name="ur_type" default="ur5e"/>
+    <!-- ================= ARGUMENTS ================= -->
     <xacro:arg name="joint_limit_params" default="$(find ur_description)/config/ur5e/joint_limits.yaml"/>
     <xacro:arg name="kinematics_params" default="$(find ur_description)/config/ur5e/default_kinematics.yaml"/>
     <xacro:arg name="physical_params" default="$(find ur_description)/config/ur5e/physical_parameters.yaml"/>
     <xacro:arg name="visual_params" default="$(find ur_description)/config/ur5e/visual_parameters.yaml"/>
+    <!-- ================= BASE WORLD ================= -->
+    <link name="world"/>
+    <!-- ================= INCLUDE UR MACRO ================= -->
+    <xacro:include filename="$(find ur_description)/urdf/ur_macro.xacro"/>
+    <!-- Disable heavy collision meshes -->
+    <xacro:property name="use_collision" value="false"/>
+    <!-- ================= WORKBENCH ================= -->
     <link name="workbench_link">
         <visual>
@@ -24,6 +29,8 @@
         <inertial>
             <mass value="100.0"/>
-            <origin xyz="0 0 0" rpy="0 0 0"/>
-            <inertia ixx="1.0" ixy="0.0" ixz="0.0" iyy="1.0" iyz="0.0" izz="1.0"/>
+            <origin xyz="0 0 0"/>
+            <inertia ixx="1.0" ixy="0.0" ixz="0.0"
+                     iyy="1.0" iyz="0.0"
+                     izz="1.0"/>
         </inertial>
     </link>
@@ -31,5 +38,7 @@
         <parent link="world"/>
         <child link="workbench_link"/>
-        <origin xyz="0 0 0.4" rpy="0 0 0"/> </joint>
+        <origin xyz="0 0 0.4"/>
+    </joint>
+    <!-- ================= ARM 1 ================= -->
     <xacro:ur_robot
         name="arm1"
@@ -39,7 +48,9 @@
         kinematics_parameters_file="$(arg kinematics_params)"
         physical_parameters_file="$(arg physical_params)"
-        visual_parameters_file="$(arg visual_params)">
-        <origin xyz="-0.6 0 0.4" rpy="0 0 0"/>
+        visual_parameters_file="$(arg visual_params)"
+        use_fake_hardware="true">
+        <origin xyz="-0.7 0 0.45" rpy="0 0 0"/>
     </xacro:ur_robot>
+    <!-- ================= ARM 2 ================= -->
     <xacro:ur_robot
         name="arm2"
@@ -49,6 +60,19 @@
         kinematics_parameters_file="$(arg kinematics_params)"
         physical_parameters_file="$(arg physical_params)"
-        visual_parameters_file="$(arg visual_params)">
-        <origin xyz="0.6 0 0.4" rpy="0 0 0"/>
+        visual_parameters_file="$(arg visual_params)"
+        use_fake_hardware="true">
+        <origin xyz="0.7 0 0.45" rpy="0 0 0"/>
     </xacro:ur_robot>
+    <!-- ================= GAZEBO SETTINGS ================= -->
+    <!-- Global physics stability -->
+    <gazebo>
+        <gravity>true</gravity>
+    </gazebo>
+    <!-- Workbench friction -->
+    <gazebo reference="workbench_link">
+        <mu1>0.5</mu1>
+        <mu2>0.5</mu2>
+        <kp>100000.0</kp>
+        <kd>1.0</kd>
+    </gazebo>
 </robot>
