Commit message: update

File: src/dual_ur5/urdf/ur5e.urdf (robot description, URDF)
Before this commit: robot ur5e_robot, 11 links, 10 joints
Links:
- removed link base_link_inertia
- link base_link: mass None -> 4.0; geometry collision mesh filename=package://dual_ur5/urdf/meshes/collision/base.stl; visual mesh filename=package://dual_ur5/urdf/meshes/visual/base.dae
Joints:
- removed joint base_link-base_link_inertia
- joint shoulder_pan_joint: parent base_link_inertia -> base_link

Commit message: added screw driver tool

File: src/dual_ur5/urdf/ur5e.urdf (robot description, URDF)
Before this commit: robot $(arg robot_name), 11 links, 10 joints
Links:
- added link housing_base_link, mass 0.1; collision cylinder length=0.05 radius=0.04; visual mesh filename=package://dual_ur5/urdf/meshes/collision/EndEffectorMountCo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 scale=0.001 0.001 0.001
- added link screw_tool_base_link, mass 0.268; collision cylinder length=0.12 radius=0.03; visual mesh filename=package://dual_ur5/urdf/meshes/collision/end_effector.stl scale=0.001 0.001 0.001
- added link screw_tool_camera_link
- added link screw_tool_tool_point
- added link screwblock_base_link, mass 0.1; collision cylinder length=0.05 radius=0.04; visual mesh filename=package://dual_ur5/urdf/meshes/collision/EndEffectorMountHo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 scale=0.001 0.001 0.001
Joints:
- added joint screw_tool_camera_joint: type fixed, parent screw_tool_base_link, child screw_tool_camera_link, origin xyz=-0.02 0 0.07989 rpy=3.141592653589793 3.141592653589793 0
- added joint screw_tool_end_effector_flange: type fixed, parent tool0, child screw_tool_base_link, origin xyz=0 0 0.01 rpy=0 0 0
- added joint screw_tool_tool_point_joint: type fixed, parent screw_tool_base_link, child screw_tool_tool_point, origin xyz=-0.0975 0 0.02 rpy=0 0 0
- added joint tool0_to_housing: type fixed, parent tool0, child housing_base_link, origin xyz=0 0 0 rpy=0 0 0
- added joint tool0_to_screwblock: type fixed, parent tool0, child screwblock_base_link, origin xyz=0 0 0 rpy=0 0 0
- joint shoulder_lift_joint: limit lower=-6.283185307179586 upper=6.283185307179586 effort=150.0 velocity=3.141592653589793 -> lower=3.141592653589793 upper=6.283185307179586 effort=150.0 velocity=3.141592653589793

Commit message: added moveit

File: src/dual_ur5/urdf/ur5e.urdf (robot description, URDF)
Before this commit: robot $(arg robot_name), 16 links, 15 joints
Links:
- removed link base
- removed link base_link
- removed link flange
- removed link forearm_link
- removed link housing_base_link
- removed link screw_tool_base_link
- removed link screw_tool_camera_link
- removed link screw_tool_tool_point
- removed link screwblock_base_link
- removed link shoulder_link
- removed link tool0
- removed link upper_arm_link
- removed link wrist_1_link
- removed link wrist_2_link
- removed link wrist_3_link
Joints:
- removed joint base_link-base_fixed_joint
- removed joint elbow_joint
- removed joint flange-tool0
- removed joint screw_tool_camera_joint
- removed joint screw_tool_end_effector_flange
- removed joint screw_tool_tool_point_joint
- removed joint shoulder_lift_joint
- removed joint shoulder_pan_joint
- removed joint tool0_to_housing
- removed joint tool0_to_screwblock
- removed joint world_joint
- removed joint wrist_1_joint
- removed joint wrist_2_joint
- removed joint wrist_3-flange
- removed joint wrist_3_joint
