Commit message: init motion planning.
Co-authored-by: Copilot <copilot@github.com>

File: src/dual_ur5/urdf/ur5e_macro.xacro (robot description, xacro)
@@ -227,44 +227,8 @@
       <child link="${prefix}tool0"/>
     </joint>
-    <joint name="${prefix}screw_tool_end_effector_flange" type="fixed">
-      <parent link="${prefix}tool0"/>
-      <child link="${prefix}screw_tool_base_link"/>
-      <origin xyz="0 0 0.01" rpy="0 0 0"/>
-    </joint>
-    <link name="${prefix}screw_tool_base_link">
-      <visual>
-        <geometry>
-          <mesh filename="package://dual_ur5/urdf/meshes/collision/end_effector.stl" scale="0.001 0.001 0.001"/>
-        </geometry>
-        <origin xyz="0 0 0" rpy="3.141592653589793 0 1.5707963267948966"/>
-      </visual>
-      <collision>
-        <geometry>
-          <cylinder radius="0.03" length="0.12"/>
-        </geometry>
-        <origin xyz="0 0 0.06" rpy="3.141592653589793 0 1.5707963267948966"/>
-      </collision>
-      <inertial>
-        <origin xyz="0 0 0" rpy="0 0 0"/>
-        <mass value="0.268"/>
-        <inertia ixx="0.0005" ixy="0.0" ixz="0.0" iyy="0.0005" iyz="0.0" izz="0.0001"/>
-      </inertial>
-    </link>
-    <link name="${prefix}screw_tool_camera_link"> </link>
-    <joint name="${prefix}screw_tool_camera_joint" type="fixed">
-        <parent link="${prefix}screw_tool_base_link"/>
-        <child link="${prefix}screw_tool_camera_link"/>
-        <origin xyz="-0.02 0 0.07989" rpy="3.141592653589793 3.141592653589793 0"/>
-    </joint>
-    <link name="${prefix}screw_tool_tool_point"> </link>
-    <joint name="${prefix}screw_tool_tool_point_joint" type="fixed">
-        <parent link="${prefix}screw_tool_base_link"/>
-        <child link="${prefix}screw_tool_tool_point"/>
-        <origin xyz="-0.0975 0 0.02" rpy="0 0 0"/>
-    </joint>
     <joint name="${prefix}tool0_to_housing" type="fixed">
       <parent link="${prefix}tool0"/>
       <child link="${prefix}housing_base_link"/>
-      <origin xyz="0 0 0" rpy="0 0 0"/>
+      <origin xyz="0 0.0 0.01" rpy="0 0 0"/>
     </joint>
     <link name="${prefix}housing_base_link">
@@ -273,5 +237,5 @@
           <mesh filename="package://dual_ur5/urdf/meshes/collision/EndEffectorMountConnectorHousing-v1.stl" scale="0.001 0.001 0.001"/>
         </geometry>
-        <origin xyz="0 0 0" rpy="1.5707963267948966 0 0"/>
+        <origin xyz="0 0 0" rpy="-1.5707963267948966 0 0"/>
       </visual>
       <collision>
@@ -279,5 +243,5 @@
           <cylinder radius="0.04" length="0.05"/>
         </geometry>
-        <origin xyz="0 0 0" rpy="1.5707963267948966 0 0"/>
+        <origin xyz="0 0 0" rpy="-1.5707963267948966 0 0"/>
       </collision>
       <inertial>
@@ -287,28 +251,85 @@
       </inertial>
     </link>
-    <joint name="${prefix}tool0_to_screwblock" type="fixed">
-      <parent link="${prefix}tool0"/>
-      <child link="${prefix}screwblock_base_link"/>
-      <origin xyz="0 0 0" rpy="0 0 0"/>
-    </joint>
-    <link name="${prefix}screwblock_base_link">
-      <visual>
-        <geometry>
-          <mesh filename="package://dual_ur5/urdf/meshes/collision/EndEffectorMountHousing_ScrewBlock-v1.stl" scale="0.001 0.001 0.001"/>
-        </geometry>
-        <origin xyz="0 0 0" rpy="3.141592653589793 0 0"/>
-      </visual>
-      <collision>
-        <geometry>
-          <cylinder radius="0.04" length="0.05"/>
-        </geometry>
-        <origin xyz="0 0 0" rpy="3.141592653589793 0 0"/>
-      </collision>
-      <inertial>
-        <origin xyz="0 0 0" rpy="0 0 0"/>
-        <mass value="0.1"/>
-        <inertia ixx="0.0005" ixy="0.0" ixz="0.0" iyy="0.0005" iyz="0.0" izz="0.0001"/>
-      </inertial>
-    </link>
+    <xacro:if value="${'$(arg end_effector)' == 'vacuum'}">
+      <link name="${prefix}vacuum_gripper">
+        <visual>
+          <geometry>
+            <mesh filename="package://dual_ur5/urdf/meshes/collision/vacuum_gripper.stl" scale="0.0001 0.0001 0.0001"/>
+          </geometry>
+          <material name="blue">
+            <color rgba="0.1 0.1 0.8 1.0"/>
+          </material>
+        </visual>
+        <collision>
+          <geometry>
+            <mesh filename="package://dual_ur5/urdf/meshes/collision/vacuum_gripper.stl" scale="0.0001 0.0001 0.0001"/>
+          </geometry>
+        </collision>
+        <inertial>
+          <mass value="0.3"/>
+          <inertia ixx="0.001" ixy="0.0" ixz="0.0" iyy="0.001" iyz="0.0" izz="0.001"/>
+        </inertial>
+      </link>
+      <joint name="${prefix}vacuum_gripper_joint" type="fixed">
+        <parent link="${prefix}housing_base_link"/>
+        <child link="${prefix}vacuum_gripper"/>
+        <origin xyz="0 0.0 0.01" rpy="0 3.1416 0"/>
+      </joint>
+    </xacro:if>
+    <xacro:if value="${'$(arg end_effector)' == 'pry_tool'}">
+      <link name="${prefix}pry_tool">
+        <visual>
+          <geometry>
+            <mesh filename="package://dual_ur5/urdf/meshes/collision/Pry_tool.stl" scale="0.0001 0.0001 0.0001"/>
+          </geometry>
+          <material name="orange">
+            <color rgba="0.8 0.4 0.1 1.0"/>
+          </material>
+        </visual>
+        <collision>
+          <geometry>
+            <mesh filename="package://dual_ur5/urdf/meshes/collision/Pry_tool.stl" scale="0.0001 0.0001 0.0001"/>
+          </geometry>
+        </collision>
+        <inertial>
+          <mass value="0.2"/>
+          <inertia ixx="0.001" ixy="0.0" ixz="0.0" iyy="0.001" iyz="0.0" izz="0.001"/>
+        </inertial>
+      </link>
+      <joint name="${prefix}pry_tool_joint" type="fixed">
+        <parent link="${prefix}housing_base_link"/>
+        <child link="${prefix}pry_tool"/>
+        <origin xyz="0 0.003 0.025" rpy="0 0 0"/>
+      </joint>
+    </xacro:if>
+    <xacro:if value="${'$(arg end_effector)' == 'screwdriver'}">
+      <link name="${prefix}screwdriver">
+        <visual>
+          <geometry>
+            <mesh filename="package://dual_ur5/urdf/meshes/collision/end_effector.stl" scale="0.001 0.001 0.001"/>
+          </geometry>
+          <origin xyz="0 0 0" rpy="3.141592653589793 0 1.5707963267948966"/>
+          <material name="silver">
+            <color rgba="0.8 0.8 0.8 1.0"/>
+          </material>
+        </visual>
+        <collision>
+          <geometry>
+            <cylinder radius="0.03" length="0.12"/>
+          </geometry>
+          <origin xyz="0 0 0.06" rpy="3.141592653589793 0 1.5707963267948966"/>
+        </collision>
+        <inertial>
+          <origin xyz="0 0 0" rpy="0 0 0"/>
+          <mass value="0.268"/>
+          <inertia ixx="0.0005" ixy="0.0" ixz="0.0" iyy="0.0005" iyz="0.0" izz="0.0001"/>
+        </inertial>
+      </link>
+      <joint name="${prefix}screwdriver_joint" type="fixed">
+        <parent link="${prefix}housing_base_link"/>
+        <child link="${prefix}screwdriver"/>
+        <origin xyz="0 0 0.01" rpy="0 0 0"/>
+      </joint>
+    </xacro:if>
     <ros2_control name="${prefix}system" type="system">
       <hardware>
